File: hardware/ymmcu-ft2232.kicad_pcb (KiCad board)
At the start: 2 copper layers, 39.1 x 28.9 mm, 51 parts, among them J1 2x7 JTAG, J2 UART, J3 JTAG, J4 PWR, J5 USB_B_Micro, J6 USB_C_Receptacle_USB2.0, U1 FT2232HL, U2 93LC56BISN, X1 XTL_4_12MHz_3225

Commit message: Ready.
Parts:
- D3: value PWRLED -> PWR
- moved J4 7.62 mm to (108.0, 59.7), turned to 180 degrees
Routing:
- net /5V0: track 20.7 -> 27.1 mm, vias 0 -> 2
- net /1V8: track 55.6 -> 53.0 mm
- net /3V3: track 105.7 -> 108.2 mm
- net /BC4_TXLED: track 12.9 -> 13.8 mm
Other:
- outline, holes or cut-outs redrawn
- board text added: "G G G G G G G"
- board text added: "NC NC TDI TDO TCK TMS 3V3"
- board text added: "TCK TDI TDO TMS"
- board text added: "TX RX"
- board text added: "YMMCU-FT2232H"
- board text removed: "ymmcu-ft2232h"
