File: hardware/ymmcu-ft2232.sch (KiCad schematic (older format))
At the start: 51 parts, among them J1 2x7 JTAG, J2 UART, J3 JTAG, J4 PWR, J5 USB_B_Micro, J6 USB_C_Receptacle_USB2.0, U1 FT2232HL, U2 93LC56BISN, X1 XTL_4_12MHz_3225

Commit message: Ready.
Parts:
- C9: Comment 3.3nF+ -> 3.3uF+
Changed lines of the file:
@@
 F 8 "C53175" H 4799 1920 50  0001 L BNN "SuppliersPartNumber"
 F 9 "" H 4799 1820 50  0001 L BNN "Notepad"
-F 10 "3.3nF+" H 5450 2650 50  0000 R CNN "Comment"
+F 10 "3.3uF+" H 5450 2650 50  0000 R CNN "Comment"
 	1    4800 2600
 	0    -1   -1   0
